File: BPEM488THD.sch (KiCad schematic (older format))
At the start: 0 parts

Commit message: Add files via upload
Other:
- note added: "De-Bug 12. via the BDM input connector."
- note added: "It consists of two boards connected together with a 36 pin terminal"
- note added: "The CPU reset and EEEM Load momentary contact switches are on \nthe auxilliary board and are accessed through holes in the enclosure \ncover."
- note added: "The auxilliary board contains the power supplies and output circuits."
- note added: "The hardware for the BPEM488 engine controller is designed to fit"
- note added: "The high current ignition and injector drivers are in a separate"
- note added: "The monitoring of the engine operating parameters and engine"
- note added: "This is a one off project and I have no formal training in electronics \nor microcontroller programming. At my age SMDs present a real \nchallenge for assembly so I have used through hole components as \nmuch as possible. No doubt there are better ways to do what I have \ndone, but if it works and is dependable, that is all I ask.\n\n"
- note added: "This sheet contains the schematics for the MC9S12XEP100 CPU,"
- note added: "This sheet contains the schematics for the inputs and the RS232."
- note added: "board."
- note added: "changes are loaded by using Dirk Heisswolf's Mini BDM Pod running"
- note added: "controller."
- note added: "enclosure as is the manually controlled idle air stepper motor"
- note added: "in the LM Heeger EAF-400 Plain extruded aluminum enclosure.\n"
- note added: "strip. The main board contains the CPU, inputs and RS232 circuits."
- note added: "the BDM connection and the pin terminal strip to the auxilliary"
- note added: "tuning is done by communicating with Tuner Studio. Program"
Changed lines of the file:
@@
 $EndDescr
 $Sheet
-S 3950 2700 700  1950
+S 2350 3100 2800 600
 U 5F09E690
 F0 "Inputs_RS232" 50
@@
 $EndSheet
 $Sheet
-S 6050 2650 700  1950
+S 6050 3100 2850 650
 U 5EF2B07F
 F0 "CPU" 50
 F1 "CPU.sch" 50
 $EndSheet
+Text Notes 6200 3350 0    50   ~ 0
+This sheet contains the schematics for the MC9S12XEP100 CPU,
+Text Notes 6200 3450 0    50   ~ 0
+the BDM connection and the pin terminal strip to the auxilliary
+Text Notes 6200 3550 0    50   ~ 0
+board.
+Text Notes 2450 3400 0    50   ~ 0
+This sheet contains the schematics for the inputs and the RS232.
+Text Notes 4200 800  0    50   ~ 0
+The hardware for the BPEM488 engine controller is designed to fit
+Text Notes 4200 900  0    50   ~ 0
+in the LM Heeger EAF-400 Plain extruded aluminum enclosure.\n
+Text Notes 4200 1000 0    50   ~ 0
+It consists of two boards connected together with a 36 pin terminal
+Text Notes 4200 1100 0    50   ~ 0
+strip. The main board contains the CPU, inputs and RS232 circuits.
+Text Notes 4200 1200 0    50   ~ 0
+The auxilliary board contains the power supplies and output circuits.
+Text Notes 4200 1300 0    50   ~ 0
+The high current ignition and injector drivers are in a separate
+Text Notes 4200 1400 0    50   ~ 0
+enclosure as is the manually controlled idle air stepper motor
+Text Notes 4200 1500 0    50   ~ 0
+controller.
+Text Notes 4200 1600 0    50   ~ 0
+The monitoring of the engine operating parameters and engine
+Text Notes 4200 1700 0    50   ~ 0
+tuning is done by communicating with Tuner Studio. Program
+Text Notes 4200 1800 0    50   ~ 0
+changes are loaded by using Dirk Heisswolf's Mini BDM Pod running
+Text Notes 4200 1900 0    50   ~ 0
+De-Bug 12. via the BDM input connector.
+Text Notes 4200 2400 0    50   ~ 0
+This is a one off project and I have no formal training in electronics \nor microcontroller programming. At my age SMDs present a real \nchallenge for assembly so I have used through hole components as \nmuch as possible. No doubt there are better ways to do what I have \ndone, but if it works and is dependable, that is all I ask.\n\n
+Text Notes 4200 2600 0    50   ~ 0
+The CPU reset and EEEM Load momentary contact switches are on \nthe auxilliary board and are accessed through holes in the enclosure \ncover.
 $EndSCHEMATC
