File: Inputs_RS232.sch (KiCad schematic (older format))
At the start: 70 parts, among them J201 DB9_Female, J202 DB25_Female, Q201 ZTX450, Q202 ZTX450, Q203 ZTX450, U201 MPXA6115AC7U, U202 4N25, U203 4N25, U204 4N25, U205 MAX232

Commit message: Add files via upload
Parts:
- J202: footprint digikey-footprints:DB15FC -> Connector_Dsub:DSUB-25_Female_Horizontal_P2.77x2.84mm_EdgePinOffset4.94mm_Housed_MountingHolesOffset7.48mm; Digikey L77SDB25S1ACH4R-ND -> AE10935-ND; Mfg L77SDB25S1ACH4R -> A-DF 25 A/KG-T2S
Connections:
- net PA0 is gone; now on net EGO: J202.1
- net +8V: now also J202.24 (P24); no longer J202.16 (P16)
- net CKP: now also J202.25 (P25); no longer J202.17 (P17)
- net CLT: now also J202.18 (P18); no longer J202.19 (P19)
- net CMP: now also J202.12; no longer J202.4
- net EFP: now also J202.5; no longer J202.10
- net EGO: no longer J202.9
- net EOP: now also J202.6; no longer J202.22 (P22)
- net Ftrm: now also J202.3; no longer J202.11
- net GND: now also J202.11, J202.20 (P20), J202.7; no longer J202.12, J202.18 (P18), J202.3
- net Itrm: now also J202.4; no longer J202.23 (P23)
- net MAP: now also J202.15 (P15); no longer J202.8
- net MAT: now also J202.17 (P17); no longer J202.7
- net PA1: now also J202.23 (P23); no longer J202.14 (P14)
- net PA3: now also J202.22 (P22); no longer J202.2
- net PA4: now also J202.9; no longer J202.15 (P15)
- net PA5: now also J202.21 (P21); no longer J202.25 (P25)
- net PA6: now also J202.8; no longer J202.13
- net PAD03in: now also J202.16 (P16); no longer J202.20 (P20)
- net PAD05: now also C206.2, R211.2; no longer C217.2, R201.1, U201.4 (Vout)
- net PAD06: now also C207.2, R212.2; no longer C206.2, R211.2
- net PAD07: now also C217.2, R201.1, U201.4 (Vout); no longer C207.2, R212.2
- net PAD12in: now also J202.2; no longer J202.24 (P24)
- net TPS: now also J202.14 (P14); no longer J202.21 (P21)
- net VDD: now also J202.19 (P19); no longer J202.6
- net VSPD: now also J202.13; no longer J202.5
- new net PA2: J202.10
Other:
- note added: "8V Gnd"
- note added: "PA4 Input\n"
- note added: "PA5 Input\n"
- note added: "PA6 Input\n"
- note added: "VDD Gnd"
- note removed: "PA4 Spare"
- note removed: "PA5 Spare"
- note removed: "PA6 Spare"
- moved on the sheet: C206, C207, C214, C215, C217, C218, R201, R211, R212, R225, R226, R227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

Commit message: Add files via upload
Parts:
- U205: value MAX232 -> MAX232EEPE+
Other:
- note added: "NOTE! The stock CMP, CKP and VSPD sensors require an 8 volt power\nsupply."
- note added: "PAD00 = +Batt = Battery Voltage\nPAD01 = CLT = Coolant Temperature\nPAD02 = MAT = Manifold Air Temperature\nPAD03 = PAD03in = Spare ADC Temperature in\nPAD04 = MAP = Manifold Absolute Pressure\nPAD05 = TPS = Throttle Position Sensor\nPAD06 = EGO = Exhaust Gas Oxygen Sensor\nPAD07 = Barometric Pressure Sensor (board mount)\nPAD08 = EOP = Engine Oil Pressure Sensor\nPAD09 = EFP = Engine Fuel Pressu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"
- note added: "PT0 = CMP = Camshaft Position Sensor\nPT1 = CKP = Crankshaft Position Sensor\nPT2 = VSPD = Vehicle Speed Sensor\nPA1 = Ignition Trim Enable Switch\nPA2 = Fuel Trim Enable Switch\nPA3 = Alarm Silence Switch\nPA4 = PA4 input spare\nPA5 = PA5 input spare\nPA6 = PA6 input spare\nPS0 = RS232 Rx\nPS1 = RS232 Tx"
Changed lines of the file:
@@
 AR Path="/5F09E690/5F0D7694" Ref="U205"  Part="1"
 F 0 "U205" H 8100 6531 50  0000 C CNN
-F 1 "MAX232" H 8100 6440 50  0000 C CNN
+F 1 "MAX232EEPE+" H 8100 6440 50  0000 C CNN
 F 2 "digikey-footprints:DIP-16_W7.62mm" H 8150 4100 50  0001 L CNN
 F 3 "https://datasheets.maximintegrated.com/en/ds/MAX202E-MAX241E.pdf" H 8100 5250 50  0001 C CNN
@@
 Wire Wire Line
 	5950 2900 6100 2900
+Text Notes 2250 4950 0    50   ~ 0
+PAD00 = +Batt = Battery Voltage\nPAD01 = CLT = Coolant Temperature\nPAD02 = MAT = Manifold Air Temperature\nPAD03 = PAD03in = Spare ADC Temperature in\nPAD04 = MAP = Manifold Absolute Pressure\nPAD05 = TPS = Throttle Position Sensor\nPAD06 = EGO = Exhaust Gas Oxygen Sensor\nPAD07 = Barometric Pressure Sensor (board mount)\nPAD08 = EOP = Engine Oil Pressure Sensor\nPAD09 = EFP = Engine Fuel Pressure Sensor\nPAD10 = Itrm = Ignition Trim Potentiometer\nPAD11 = Ftrm = Fuel Trim Potentiometer\nPAD12 = PAD12in = Spare ADC in
+Text Notes 4650 4800 0    50   ~ 0
+PT0 = CMP = Camshaft Position Sensor\nPT1 = CKP = Crankshaft Position Sensor\nPT2 = VSPD = Vehicle Speed Sensor\nPA1 = Ignition Trim Enable Switch\nPA2 = Fuel Trim Enable Switch\nPA3 = Alarm Silence Switch\nPA4 = PA4 input spare\nPA5 = PA5 input spare\nPA6 = PA6 input spare\nPS0 = RS232 Rx\nPS1 = RS232 Tx
+Text Notes 4400 1050 0    50   ~ 0
+NOTE! The stock CMP, CKP and VSPD sensors require an 8 volt power\nsupply.
 $EndSCHEMATC

Commit message: Add files via upload
Parts:
- removed C215: 0.22uF, Capacitor_THT:C_Disc_D5.0mm_W2.5mm_P2.50mm, symbol Device:C
- added R228: 1Meg, Resistor_THT:R_Axial_DIN0207_L6.3mm_D2.5mm_P10.16mm_Horizontal, symbol Device:R
- C205, C206, C207, C208, C220, C221, C222: value 0.001uF -> 0.22uF; footprint Capacitor_THT:C_Disc_D3.8mm_W2.6mm_P2.50mm -> Capacitor_THT:C_Disc_D5.0mm_W2.5mm_P2.50mm; Digikey 399-4144-ND -> 399-4289-ND; Mfg C315C102K1R5TA -> C320C224M5U5TA
- C213, C214, C216, C223, C224, C225, C226: value 0.22uF -> 0.001uF; footprint Capacitor_THT:C_Disc_D5.0mm_W2.5mm_P2.50mm -> Capacitor_THT:C_Disc_D3.8mm_W2.6mm_P2.50mm; Digikey 399-4289-ND -> 399-4144-ND; Mfg C320C224M5U5TA -> C315C102K1R5TA
- C219: value 0.001uF -> 0.22uF; footprint Capacitor_THT:C_Disc_D3.8mm_W2.6mm_P2.50mm -> Capacitor_THT:C_Disc_D5.0mm_W2.5mm_P2.50mm; Digikey (none) -> 399-4289-ND; Mfg (none) -> C320C224M5U5TA
- C230, C231, C232, C233: value 0.22uF -> 1.0uF; footprint Capacitor_THT:C_Disc_D5.0mm_W2.5mm_P2.50mm -> Capacitor_THT:C_Disc_D3.8mm_W2.6mm_P2.50mm; Digikey 399-4289-ND -> 399-9714-ND; Mfg C320C224M5U5TA -> C315C105K3R5TA
- J201: footprint digikey-footprints:DB9Fem -> Connector_Dsub:DSUB-9_Female_Horizontal_P2.77x2.84mm_EdgePinOffset9.90mm_Housed_MountingHolesOffset11.32mm
- J202: footprint Connector_Dsub:DSUB-25_Female_Horizontal_P2.77x2.84mm_EdgePinOffset4.94mm_Housed_MountingHolesOffset7.48mm -> Connector_Dsub:DSUB-25_Female_Horizontal_P2.77x2.84mm_EdgePinOffset7.70mm_Housed_MountingHolesOffset9.12mm
- R201: value 51K -> 51.1K; Digikey (none) -> 51.0KXBK-ND; Mfg (none) -> MFR-25FBF52-51K1
- R202: Digikey (none) -> 49.9KXBK-ND; Mfg (none) -> MFR-25FBF52-49K9
- R203, R205, R207, R209, R210, R211, R212, R213, R215, R216, R217, R218, R219, R220, R221, R222, R223, R224: Digikey (none) -> 1.00KXBK-ND; Mfg (none) -> MFR-25FBF52-1K
- R204, R206, R208: Digikey (none) -> 6.98KXBK-ND; Mfg (none) -> MFR-25FBF52-6K98
- R214: Digikey (none) -> 10.0KXBK-ND; Mfg (none) -> MFR-25FBF52-10K
- R225, R226, R227: value 1.5K -> 200R; Digikey (none) -> 200XBK-ND; Mfg (none) -> MFR-25FBF52-200R
Connections:
- net EGO: now also R228.1
- net GND: now also R228.2; no longer J201.9
- net VDD: now also J201.9

Commit message: Add files via upload
Parts:
- removed C227, C228, C229: 1.0uF, Capacitor_THT:C_Disc_D3.8mm_W2.6mm_P2.50mm, symbol Device:C
Connections:
- net GND: now also U202.2, U203.2, U204.2; no longer U202.4, U203.4, U204.4
- net PT0: now also R219.1, R222.2
- net PT1: now also R220.1, R223.2
- net PT2: now also R221.1, R224.2
- net VDD: now also U202.5, U203.5, U204.5; no longer U202.1, U203.1, U204.1
- net at Q202.2 (B), R220.2: now also U203.4; no longer U203.2
- net at R226.2: now also U203.1; no longer U203.5
- net at Q203.2 (B), R221.2: now also U204.4; no longer U204.2
- net at R227.2: now also U204.1; no longer U204.5
- net at Q201.2 (B), R219.2: now also U202.4; no longer U202.2
- net at R225.2: now also U202.1; no longer U202.5
Other:
- note added: "8V signal goes low at trigger point"
- note added: "8V square wave 8000 pp Mile"
- note added: "High at trigger"
- moved on the sheet: Q202, Q203, R220, R221, R223, R224, R226, R227, U203, U204
