File: BPEM488THD.kicad_pcb (KiCad board)
At the start: 2 copper layers, 152.4 x 101.6 mm, 90 parts, among them J201 DB9_Female, J202 DB25_Female, J301 Molex+Microfit3-Dual4-90, J302 Conn_02x18_Odd_Even, Q201 ZTX450, Q202 ZTX450, Q203 ZTX450, U201 MPXA6115AC7U, U202 4N25, U203 4N25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

Commit message: Add files via upload
Parts:
- moved C217 5.08 mm to (184.8, 137.9)
- moved C218 5.08 mm to (182.2, 143.0)
- moved R201 5.08 mm to (182.2, 132.9)
- moved U201 5.08 mm to (179.7, 145.6)
- moved J201 2.32 mm to (209.5, 133.5)
- moved C230 1.27 mm to (192.0, 129.0)
- moved C231 1.27 mm to (192.0, 136.7)
- moved J302 1.27 mm to (137.2, 78.7)
- moved U205 1.27 mm to (195.8, 126.5)
- moved C232 1.27 mm to (186.9, 129.0)
- moved C233 1.27 mm to (190.8, 140.5)
Connections:
- J302 pad 13: /CPU/PK5 -> GND
- J302 pad 15: /CPU/PK4 -> GND
- J302 pad 17: /CPU/PB0 -> GND
- J302 pad 19: /CPU/PB1 -> GND
- J302 pad 21: /CPU/PB2 -> VDD
- J302 pad 23: /CPU/PB3 -> +BATT
- J302 pad 25: /CPU/PB4 -> /CPU/RESET
- J302 pad 26: +8V -> /CPU/PK5
- J302 pad 27: /CPU/PB5 -> /CPU/PA0
- J302 pad 28: VDD -> /CPU/PK4
- J302 pad 29: /CPU/PB6 -> +8V
- J302 pad 30: GND -> /CPU/PB0
- J302 pad 31: /CPU/RESET -> /CPU/PB6
- J302 pad 32: GND -> /CPU/PB1
- J302 pad 33: +BATT -> /CPU/PB5
- J302 pad 34: /CPU/PA0 -> /CPU/PB2
- J302 pad 35: GND -> /CPU/PB4
- J302 pad 36: GND -> /CPU/PB3
Routing:
- net VDD: track 199.5 -> 553.8 mm, vias 3 -> 5
- net GND: track 299.8 -> 85.9 mm, vias 9 -> 10
- net Net-(J301-Pad1): track 20.7 -> 186.2 mm, vias 0 -> 2
- net /CPU/RESET: track 26.6 -> 190.6 mm, vias 0 -> 2
- net PA2: track 65.3 -> 202.0 mm
- net PAD08: track 41.6 -> 176.1 mm
- net PA1: track 66.7 -> 198.9 mm
- net PA3: track 70.4 -> 202.5 mm
- net PA4: track 69.3 -> 201.2 mm
- net +8V: track 37.1 -> 168.7 mm, vias 0 -> 1
- net PA5: track 74.4 -> 205.6 mm
- net PA6: track 73.5 -> 204.3 mm
- net PAD09: track 44.3 -> 168.1 mm
- net PAD10: track 47.0 -> 159.3 mm
- net PAD01: track 43.0 -> 154.6 mm
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- added copper zone on B.Cu, net GND
- added copper zone on F.Cu, net GND
Other:
- outline, holes or cut-outs redrawn
- net class 1 amp added: clearance 0.3, trace_width 0.3, via_dia 0.8, via_drill 0.4
- net class 1.5 amp added: clearance 0.35052, trace_width 0.508, via_dia 0.8, via_drill 0.4
- net class 2 amp added: clearance 0.35052, trace_width 0.762, via_dia 0.8, via_drill 0.4
- net class 2.5 amp added: clearance 0.35052, trace_width 1.016, via_dia 0.8, via_drill 0.4
- net class 3 amp added: clearance 0.35052, trace_width 1.27, via_dia 0.8, via_drill 0.4
- net class Default: clearance 0.3 -> 0.2; trace_width 0.3 -> 0.25
- rule trace_clearance: 0.3 -> 0.2

Commit message: Add files via upload
Parts:
- removed C215: 0.22uF, Capacitor_THT:C_Disc_D5.0mm_W2.5mm_P2.50mm
- added R228: 1Meg, Resistor_THT:R_Axial_DIN0207_L6.3mm_D2.5mm_P10.16mm_Horizontal, F.Cu at (83.8, 129.5)
- C205, C206, C207, C208, C219, C220, C221, C222: value 0.001uF -> 0.22uF; footprint Capacitor_THT:C_Disc_D3.8mm_W2.6mm_P2.50mm -> Capacitor_THT:C_Disc_D5.0mm_W2.5mm_P2.50mm
- C213, C214, C216, C223, C224, C225, C226: value 0.22uF -> 0.001uF; footprint Capacitor_THT:C_Disc_D5.0mm_W2.5mm_P2.50mm -> Capacitor_THT:C_Disc_D3.8mm_W2.6mm_P2.50mm
- C230, C231, C232, C233: value 0.22uF -> 1.0uF; footprint Capacitor_THT:C_Disc_D5.0mm_W2.5mm_P2.50mm -> Capacitor_THT:C_Disc_D3.8mm_W2.6mm_P2.50mm
- J201: footprint digikey-footprints:DB9Fem -> Connector_Dsub:DSUB-9_Female_Horizontal_P2.77x2.84mm_EdgePinOffset9.90mm_Housed_MountingHolesOffset11.32mm
- J202: footprint Connector_Dsub:DSUB-25_Female_Horizontal_P2.77x2.84mm_EdgePinOffset4.94mm_Housed_MountingHolesOffset7.48mm -> Connector_Dsub:DSUB-25_Female_Horizontal_P2.77x2.84mm_EdgePinOffset7.70mm_Housed_MountingHolesOffset9.12mm
- R201: value 51K -> 51.1K
- R225, R226, R227: value 1.5K -> 200R
- U205: value MAX232 -> MAX232EEPE+
- moved C207 14.6 mm to (101.6, 138.8), turned to 180 degrees
- moved C232 11.7 mm to (196.2, 121.9)
- moved J201 7.08 mm to (206.4, 127.2), turned to 90 degrees
- moved C233 4.58 mm to (189.2, 144.8), turned to 90 degrees
- moved C217 3.05 mm to (182.9, 140.3), turned to 90 degrees
- moved C231 2.84 mm to (189.2, 137.2)
- moved U205 2.84 mm to (193.0, 127.0)
- moved C230 2.84 mm to (189.2, 129.5)
- moved R201 2.77 mm to (179.7, 134.0)
- moved C214 1.27 mm to (101.6, 129.5)
- moved R205 1.27 mm to (99.1, 83.8)
- moved R207 1.27 mm to (99.1, 96.5)
- moved R209 1.27 mm to (99.1, 109.2)
- moved C206 1.27 mm to (106.7, 129.5)
- moved J202 1.18 mm to (70.5, 114.0)
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Connections:
- J201 pad 9: GND -> VDD
Routing:
- net Net-(C232-Pad1): track 18.8 -> 9.23 mm
- net GND: track 85.9 -> 80.8 mm, vias 10 -> 53
- net VDD: track 553.8 -> 558.4 mm, vias 5 -> 3
- net PAD06: track 139.9 -> 136.0 mm
- net /Inputs_RS232/VSPD: track 17.5 -> 19.7 mm
- net PS1: track 62.8 -> 64.9 mm, vias 0 -> 1
- net PS0: track 61.1 -> 63.2 mm, vias 1 -> 2
- net Net-(C233-Pad2): track 3.11 -> 4.88 mm
- net PAD07: track 47.0 -> 48.5 mm
- net Net-(J201-Pad3): track 5.02 -> 6.51 mm
- net Net-(J201-Pad2): track 5.26 -> 6.61 mm
- net /Inputs_RS232/CKP: track 38.9 -> 40.2 mm
- net PA4: track 201.2 -> 202.6 mm
- net /Inputs_RS232/CMP: track 64.5 -> 65.8 mm
- net /Inputs_RS232/CLT: track 47.4 -> 48.6 mm
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Other:
- board text added: "BPEM488 TDH Designed by Robert Hiebert 7-18-20"

Commit message: Add files via upload
Parts:
- removed C227, C228, C229: 1.0uF, Capacitor_THT:C_Disc_D3.8mm_W2.6mm_P2.50mm
- moved U203 9.16 mm to (108.0, 59.7), turned to 0 degrees
- moved U204 9.16 mm to (80.0, 59.7), turned to 0 degrees
- moved U202 9.12 mm to (135.9, 59.8), turned to 0 degrees
Connections:
- R219 pad 1: Net-(R219-Pad1) -> PT0
- R220 pad 1: Net-(R220-Pad1) -> PT1
- R221 pad 1: Net-(R221-Pad1) -> PT2
- R222 pad 2: Net-(R219-Pad1) -> PT0
- R223 pad 2: Net-(R220-Pad1) -> PT1
- R224 pad 2: Net-(R221-Pad1) -> PT2
- R225 pad 2: Net-(C227-Pad2) -> Net-(R225-Pad2)
- R226 pad 2: Net-(C228-Pad2) -> Net-(R226-Pad2)
- R227 pad 2: Net-(C229-Pad2) -> Net-(R227-Pad2)
- U202 pad 1: VDD -> Net-(R225-Pad2)
- U202 pad 2: Net-(Q201-Pad2) -> GND
- U202 pad 4: GND -> Net-(Q201-Pad2)
- U202 pad 5: Net-(C227-Pad2) -> VDD
- U203 pad 1: VDD -> Net-(R226-Pad2)
- U203 pad 2: Net-(Q202-Pad2) -> GND
- U203 pad 4: GND -> Net-(Q202-Pad2)
- U203 pad 5: Net-(C228-Pad2) -> VDD
- U204 pad 1: VDD -> Net-(R227-Pad2)
- U204 pad 2: Net-(Q203-Pad2) -> GND
- U204 pad 4: GND -> Net-(Q203-Pad2)
- U204 pad 5: Net-(C229-Pad2) -> VDD
Routing:
- net PT1: track 90.3 -> 104.0 mm, vias 4 -> 2
- net PT0: track 61.9 -> 75.3 mm
- net VDD: track 558.4 -> 570.9 mm
- net PT2: track 118.2 -> 130.6 mm, vias 6 -> 2
- net Net-(C227-Pad2): track 7.61 -> 0.00 mm
- net Net-(C229-Pad2): track 7.22 -> 0.00 mm
- net Net-(C228-Pad2): track 7.22 -> 0.00 mm
- net Net-(R227-Pad2): track 0.00 -> 6.68 mm
- net Net-(R226-Pad2): track 0.00 -> 6.52 mm
- net Net-(R225-Pad2): track 0.00 -> 6.44 mm
- net Net-(Q203-Pad2): track 17.9 -> 20.6 mm
- net Net-(R221-Pad1): track 2.70 -> 0.00 mm
- net Net-(R220-Pad1): track 2.54 -> 0.00 mm
- net Net-(R219-Pad1): track 2.54 -> 0.00 mm
- net Net-(Q202-Pad2): track 18.0 -> 19.2 mm
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
Commit message: Add files via upload
Routing:
- net GND: vias 46 -> 126
- net (no net): vias 1 -> 0
